Commit message: Correct myCobot JN assembly mass in URDFs

File: src/arc_mycobot/assets/robots/urdf/mycobot_280_jn_camera_gripper.urdf (robot description, URDF)
Before this commit: robot mycobot_280_jn_adaptive_gripper_camera_gripper, 19 links, 18 joints
Links:
- link camera_flange: mass None -> 0.060000
- link gripper_base: mass 0.070000 -> 0.062000
- link joint1: mass 0.240000 -> 0.420000

File: src/arc_mycobot/assets/robots/urdf/mycobot_280_jn_camera_gripper_parallel.urdf (robot description, URDF)
Before this commit: robot mycobot_280_jn_camera_gripper_parallel, 19 links, 18 joints
Links:
- link camera_flange: mass None -> 0.060000
- link gripper_base: mass 0.070000 -> 0.062000
- link joint1: mass 0.240000 -> 0.420000

Commit message: Train gravity-on randomized hand-centering policy

File: src/arc_mycobot/assets/robots/urdf/mycobot_280_jn_camera_gripper.urdf (robot description, URDF)
Before this commit: robot mycobot_280_jn_adaptive_gripper_camera_gripper, 19 links, 18 joints
Links:
- link camera_link: mass None -> 0.000100
- link camera_mount: mass None -> 0.000100
- link tcp: mass None -> 0.000100
- link tool_mount: mass None -> 0.000100

File: src/arc_mycobot/assets/robots/urdf/mycobot_280_jn_camera_gripper_parallel.urdf (robot description, URDF)
Before this commit: robot mycobot_280_jn_camera_gripper_parallel, 19 links, 18 joints
Links:
- link camera_link: mass None -> 0.000100
- link camera_mount: mass None -> 0.000100
- link tcp: mass None -> 0.000100
- link tool_mount: mass None -> 0.000100
